File: cookbook/kicad-pcb/media/data/mutants/drill_no_tools/555-blinker.kicad_pcb (KiCad board)
At the start: 2 copper layers, 40 x 30 mm, 8 parts, among them J1 Conn_01x02, U1 NE555

Commit message: wip: agent demo-kicad-pcb-harden3 (timeout)
Connections:
- D1 pad 1: LED -> GND
- D1 pad 2: GND -> LED
Routing:
- net LED: track 8.01 -> 6.27 mm
